Commit message: update

File: omron_hardware_interface/urdf/omron.ros2_control.xacro (robot description, xacro)
@@ -1,9 +1,10 @@
 <?xml version="1.0"?>
 <robot xmlns:xacro="http://www.ros.org/wiki/xacro">
-    <xacro:macro name="omron_aria" params="name">
+    <xacro:macro name="omron_aria" params="name
+                                           use_fake_hardware">
 <!--      <xacro:property name="initial_positions" value="${load_yaml(initial_positions_file)['initial_positions']}"/>-->
       <xacro:arg name="use_fake_hardware" default="false"/>
       <ros2_control name="${name}" type="system">
-        <xacro:if value="$(arg use_fake_hardware)">
+        <xacro:if value="${use_fake_hardware}">
           <hardware>
               <!-- By default, set up controllers for simulation. This won't work on real hardware -->
@@ -11,8 +12,8 @@
           </hardware>
         </xacro:if>
-        <xacro:unless value="$(arg use_fake_hardware)">
+        <xacro:unless value="${use_fake_hardware}">
           <hardware>
             <plugin>omron/OmronAria</plugin>
-            <param name="update_frequency">50</param>
+            <param name="update_frequency">500</param>
             <param name="prefix">omron_base</param>
             <param name="ip_address">192.168.1.32</param>
