Commit message: ld60 height

File: urdf/LD60.xacro (robot description, xacro)
@@ -17,5 +17,5 @@
     <link name="${prefix}base_link_omron">
       <visual>
-        <origin xyz="0 0 0.2" rpy="${M_PI/2} 0 ${M_PI/2}" />
+        <origin xyz="0 0 0.19" rpy="${M_PI/2} 0 ${M_PI/2}" />
         <geometry>
           <mesh filename="file://$(find omron_description)//mesh/LD60.stl"/>
@@ -26,5 +26,5 @@
       </visual>
       <collision>
-        <origin xyz="0 0 0.2" rpy="${M_PI/2} 0 ${M_PI/2}" />
+        <origin xyz="0 0 0.19" rpy="${M_PI/2} 0 ${M_PI/2}" />
         <geometry>
           <mesh filename="file://$(find omron_description)//mesh/LD60.stl"/>
