Commit message: xacro

File: omron_description/urdf/LD60.xacro (robot description, xacro)
@@ -6,5 +6,5 @@
   <xacro:property name="base_y_size" value="0.55" />
   <xacro:property name="base_z_size" value="0.35" />
-  <xacro:macro name="LD60" params="prefix *origin">
+  <xacro:macro name="LD60" params="prefix use_map">
     <!-- Base footprint is on the ground under the robot -->
     <!-- <link name="${prefix}base_footprint">
@@ -15,5 +15,6 @@
     </link>   -->
     <!-- Base link is the center of the robot's bottom plate -->
-    <link name="${prefix}base_link_omron">
+    <!-- <link name="${prefix}base_link_omron"> -->
+    <link name="${prefix}base_link">
       <visual>
         <origin xyz="0 0 0.19" rpy="${M_PI/2} 0 ${M_PI/2}" />
@@ -39,9 +40,23 @@
       </inertial>
     </link>
-    <joint name="${prefix}base_footprint_joint" type="fixed">
+    <!-- <joint name="${prefix}base_footprint_joint" type="fixed">
       <xacro:insert_block name="origin"/>
       <parent link="${prefix}base_link" />
       <child link="${prefix}base_link_omron" />
-    </joint>
+    </joint> -->
+    <xacro:if value="${use_map}">
+      <link name="${prefix}map"/>
+      <link name="${prefix}odom"/>
+      <joint name="map_to_odom" type="fixed">
+        <parent link="${prefix}map"/>
+        <child  link="${prefix}odom"/>
+        <!-- <axis xyz="0.0 0.0 1.0"/> -->
+      </joint>
+      <joint name="odom_to_base_link" type="planar">
+        <parent link="${prefix}odom"/>
+        <child  link="${prefix}base_link"/>
+        <axis xyz="0.0 0.0 1.0"/>
+      </joint>
+    </xacro:if>
   </xacro:macro>
 </robot>

Commit message: changed urdf

File: omron_description/urdf/LD60.xacro (robot description, xacro)
@@ -6,15 +6,8 @@
   <xacro:property name="base_y_size" value="0.55" />
   <xacro:property name="base_z_size" value="0.35" />
-  <xacro:macro name="LD60" params="prefix use_map">
+  <xacro:macro name="LD60" params="name">
     <!-- Base footprint is on the ground under the robot -->
-    <!-- <link name="${prefix}base_footprint">
-      <inertial>
-          <mass value="1000" />
-          <inertia ixx="0.001" ixy="0.01" ixz="0.01" iyy="0.001" iyz="0.01" izz="0.001" />
-      </inertial>
-    </link>   -->
-    <!-- Base link is the center of the robot's bottom plate -->
-    <!-- <link name="${prefix}base_link_omron"> -->
-    <link name="${prefix}base_link">
+    <link name="${name}mount_frame"/>
+    <link name="${name}base_footprint">
       <visual>
         <origin xyz="0 0 0.19" rpy="${M_PI/2} 0 ${M_PI/2}" />
@@ -40,23 +33,9 @@
       </inertial>
     </link>
-    <!-- <joint name="${prefix}base_footprint_joint" type="fixed">
-      <xacro:insert_block name="origin"/>
-      <parent link="${prefix}base_link" />
-      <child link="${prefix}base_link_omron" />
-    </joint> -->
-    <xacro:if value="${use_map}">
-      <link name="${prefix}map"/>
-      <link name="${prefix}odom"/>
-      <joint name="map_to_odom" type="fixed">
-        <parent link="${prefix}map"/>
-        <child  link="${prefix}odom"/>
-        <!-- <axis xyz="0.0 0.0 1.0"/> -->
-      </joint>
-      <joint name="odom_to_base_link" type="planar">
-        <parent link="${prefix}odom"/>
-        <child  link="${prefix}base_link"/>
-        <axis xyz="0.0 0.0 1.0"/>
-      </joint>
-    </xacro:if>
+    <joint name="${name}footprint_to_mount_joint" type="fixed">
+      <parent link="${name}base_footprint"/>
+      <child link="${name}mount_frame"/>
+      <origin xyz="0 0 0.38"/>
+    </joint>
   </xacro:macro>
 </robot>

File: omron_description/urdf/system.urdf.xacro (robot description, xacro)
@@ -3,5 +3,5 @@
   <xacro:arg name="use_fake_hardware" default="true"/>
   <xacro:include filename="$(find omron_description)/urdf/LD60.xacro"/>
-  <xacro:LD60 prefix="" use_map="$(arg use_fake_hardware)"/>
+  <xacro:LD60 name="omron/"/>
   <xacro:include filename="$(find omron_hardware_interface)/urdf/omron.ros2_control.xacro"/>
   <xacro:omron_aria name="omron_aria" use_fake_hardware="$(arg use_fake_hardware)"/>

Commit message: urdf

File: omron_description/urdf/LD60.xacro (robot description, xacro)
@@ -13,5 +13,5 @@
         <origin xyz="0 0 0.19" rpy="${M_PI/2} 0 ${M_PI/2}" />
         <geometry>
-          <mesh filename="file://$(find omron_description)//mesh/LD60.stl"/>
+          <mesh filename="package://omron_description/mesh/LD60.stl"/>
         </geometry>
         <material name="Gray">
@@ -22,5 +22,5 @@
         <origin xyz="0 0 0.19" rpy="${M_PI/2} 0 ${M_PI/2}" />
         <geometry>
-          <mesh filename="file://$(find omron_description)//mesh/LD60.stl"/>
+          <mesh filename="package://omron_description/mesh/LD60.stl"/>
         </geometry>
         <material name="Gray">
